File: 555_Timer_Clock.kicad_pcb (KiCad board)
At the start: 2 copper layers, 39 x 25 mm, 13 parts, among them J2 CLK_Out, U1 ICM7555xB

Commit message: update PCB
Parts:
- added J1: +5V, my_footprints:Terminal_Block_5mm, F.Cu at (102.1, 72.2)
- added SW1: Trigger, my_footprints:slide_switch_2.54mm, F.Cu at (123.0, 81.9)
- added SW2: RST, my_footprints:tact_switch_5mm, F.Cu at (112.8, 80.9)
Routing:
- net GND: track 0.00 -> 83.3 mm, vias 0 -> 2
- net /+5V: track 0.00 -> 38.4 mm
- net /Trigger: track 0.00 -> 36.8 mm
- net /CLK_Out: track 0.00 -> 27.9 mm, vias 0 -> 1
- net /RST: track 0.00 -> 19.2 mm
- net Net-(U1-DISCH): track 0.00 -> 14.2 mm
- net Net-(U1-CONT): track 0.00 -> 9.10 mm
- net Net-(D1-K): track 0.00 -> 8.44 mm
Other:
- board text added: "DE ASIS"
